File: PCB/Hangneigungssensor.kicad_pcb (KiCad board)
At the start: 2 copper layers, 53 x 19 mm, 11 parts, among them IC1 MC3632, SW1 PTS636, U1 ATtiny424, U2 BU91796, U3 LCD-DE117

Commit message: Improved annotation
Parts:
- BT1: value CR1625 -> CR1225
- renumbered R4 to R1, R5 to R2, IC1 to U2, U2 to U3, U3 to U4
Changed lines of the file:
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@@
   (general
     (thickness 1.6)
-    (drawings 26)
+    (drawings 24)
     (tracks 286)
     (zones 0)
@@
     (0 F.Cu signal hide)
     (31 B.Cu signal hide)
-    (32 B.Adhes user hide)
-    (33 F.Adhes user hide)
-    (34 B.Paste user)
-    (35 F.Paste user)
+    (32 B.Adhes user)
+    (33 F.Adhes user)
+    (34 B.Paste user hide)
+    (35 F.Paste user hide)
     (36 B.SilkS user)
-    (37 F.SilkS user)
+    (37 F.SilkS user hide)
     (38 B.Mask user)
-    (39 F.Mask user)
+    (39 F.Mask user hide)
     (40 Dwgs.User user)
     (41 Cmts.User user hide)
-    (42 Eco1.User user hide)
-    (43 Eco2.User user hide)
+    (42 Eco1.User user)
+    (43 Eco2.User user)
     (44 Edge.Cuts user)
-    (45 Margin user hide)
+    (45 Margin user)
     (46 B.CrtYd user hide)
     (47 F.CrtYd user hide)
     (48 B.Fab user)
-    (49 F.Fab user)
+    (49 F.Fab user hide)
   )
   (setup
@@
     (add_net "Net-(SW1-Pad2)")
     (add_net "Net-(U1-Pad11)")
+    (add_net "Net-(U1-Pad12)")
+    (add_net "Net-(U1-Pad13)")
+    (add_net "Net-(U1-Pad2)")
+    (add_net "Net-(U1-Pad5)")
+    (add_net "Net-(U1-Pad6)")
+    (add_net "Net-(U2-Pad11)")
+    (add_net "Net-(U2-Pad5)")
+    (add_net "Net-(U2-Pad6)")
+    (add_net "Net-(U2-Pad8)")
+    (add_net "Net-(U3-Pad20)")
+    (add_net "Net-(U3-Pad21)")
+    (add_net "Net-(U3-Pad22)")
+    (add_net "Net-(U3-Pad6)")
+    (add_net "Net-(U3-Pad7)")
+    (add_net "Net-(U3-Pad8)")
+    (add_net "Net-(U3-Pad9)")
     (add_net RESET)
     (add_net SCL)
@@
     (tags resistor)
     (attr smd)
-    (fp_text reference R5 (at 2.664 -0.006) (layer B.SilkS)
+    (fp_text reference R2 (at 2.664 -0.006) (layer B.SilkS)
       (effects (font (size 1 1) (thickness 0.15)) (justify mirror))
     )
@@
   (module 1My_Library:LCD_4x7 (layer F.Cu)
     (at 130.5 106.5)
-    (fp_text reference U3 (at 13.5 4 180) (layer F.SilkS)
+    (fp_text reference U4 (at 13.5 4 180) (layer F.SilkS)
       (effects (font (size 1 1) (thickness 0.15)))
     )
@@
       (effects (font (size 1 1) (thickness 0.15)))
     )
-    (fp_text value CR1625 (at 1.5 -0.352) (layer F.Fab)
+    (fp_text value CR1225 (at 1.5 -0.352) (layer F.Fab)
       (effects (font (size 1 1) (thickness 0.15)))
     )
@@
     (at 124.75 106.582 180)
     (attr smd)
-    (fp_text reference U2 (at 7.747 0.127 90) (layer B.SilkS)
+    (fp_text reference U3 (at 7.747 0.127 90) (layer B.SilkS)
       (effects (font (size 1 1) (thickness 0.15)) (justify mirror))
     )
@@
     (tags "lga land grid array")
     (attr smd)
-    (fp_text reference IC1 (at 2.536 0.1275) (layer B.SilkS)
+    (fp_text reference U2 (at 2.536 0.1275) (layer B.SilkS)
       (effects (font (size 1 1) (thickness 0.15)) (justify mirror))
     )
@@
     (tags resistor)
     (attr smd)
-    (fp_text reference R4 (at 2.664 -0.038 180) (layer B.SilkS)
+    (fp_text reference R1 (at 2.664 -0.038 180) (layer B.SilkS)
       (effects (font (size 1 1) (thickness 0.15)) (justify mirror))
     )
@@
     )
   )
-  (dimension 25.5 (width 0.12) (layer B.SilkS)
-    (gr_text "25,500 mm" (at 117.75 122.27) (layer B.SilkS)
-      (effects (font (size 1 1) (thickness 0.15)))
-    )
-    (feature1 (pts (xy 105 106.5) (xy 105 121.586421)))
-    (feature2 (pts (xy 130.5 106.5) (xy 130.5 121.586421)))
-    (crossbar (pts (xy 130.5 121) (xy 105 121)))
-    (arrow1a (pts (xy 105 121) (xy 106.126504 120.413579)))
-    (arrow1b (pts (xy 105 121) (xy 106.126504 121.586421)))
-    (arrow2a (pts (xy 130.5 121) (xy 129.373496 120.413579)))
-    (arrow2b (pts (xy 130.5 121) (xy 129.373496 121.586421)))
-  )
-  (dimension 27.5 (width 0.12) (layer B.SilkS)
-    (gr_text "27,500 mm" (at 144.25 122.27) (layer B.SilkS)
-      (effects (font (size 1 1) (thickness 0.15)))
-    )
-    (feature1 (pts (xy 158 106.5) (xy 158 121.586421)))
-    (feature2 (pts (xy 130.5 106.5) (xy 130.5 121.586421)))
-    (crossbar (pts (xy 130.5 121) (xy 158 121)))
-    (arrow1a (pts (xy 158 121) (xy 156.873496 121.586421)))
-    (arrow1b (pts (xy 158 121) (xy 156.873496 120.413579)))
-    (arrow2a (pts (xy 130.5 121) (xy 131.626504 121.586421)))
-    (arrow2b (pts (xy 130.5 121) (xy 131.626504 120.413579)))
-  )
-  (dimension 10.5 (width 0.12) (layer F.SilkS)
-    (gr_text "10,500 mm" (at 162.27 106.75 270) (layer F.SilkS)
+  (dimension 10.5 (width 0.12) (layer Eco1.User)
+    (gr_text "10,500 mm" (at 162.27 106.75 270) (layer Eco1.User)
       (effects (font (size 1 1) (thickness 0.15)))
     )
@@
     (arrow2b (pts (xy 161 101.5) (xy 161.586421 102.626504)))
   )
-  (dimension 19 (width 0.12) (layer F.SilkS)
-    (gr_text "19,000 mm" (at 98.73 106.5 270) (layer F.SilkS)
+  (dimension 19 (width 0.12) (layer Eco1.User)
+    (gr_text "19,000 mm" (at 98.73 106.5 270) (layer Eco1.User)
       (effects (font (size 1 1) (thickness 0.15)))
     )
@@
     (arrow2b (pts (xy 100 97) (xy 100.586421 98.126504)))
   )
-  (dimension 53 (width 0.12) (layer F.SilkS)
-    (gr_text "53,000 mm" (at 131.5 91.73) (layer F.SilkS)
-      (effects (font (size 1 1) (thickness 0.15)))
-    )
+  (dimension 53 (width 0.12) (layer Eco1.User)
+    (gr_text "53,000 mm" (at 131.5 91.73) (layer Eco1.User)
+      (effects (font (size 1 1) (thickness 0.15)))
+    )
